File: hardware/fl11/fl11.kicad_sch (KiCad schematic)
At the start: 77 parts, among them J1 USB-C 16P, J2_1 TOUCH_SENSE, J2_2 GND, J3_1 TOUCH_SENSE, J3_2 GND, J4_1 5V, J4_2 3V3, J4_3 GND, J4_4 SIG, Q1 AO3401A, SW1 BOOT, U1 ESP32-C3-MINI-1-N4, U2 SN74AHCT1G125, U3 AP2112K-3.3, U4 USBLC6-2SC6

Commit message: FL-11 rev I: a TTP223 module replaces the etched sensor
This is the biggest simplification in the design. A TTP223-class module plugs
into J4 in IO / VCC / GND order and does the sensing, which deletes the comb
electrodes, the snap-off pad section, the break line, the webs, both bridges,
and R10's 4.7M -- the thinnest-stock line on the BOM, now a 100k that was
already there. It also deletes section 7.5's entire uncertainty: the
charge-time measurement, the per-unit threshold, the overlay dependence, and
the note calling touch the least-certain subsystem in the design. touch.py
becomes a digital read.

VCC is 3V3 and not 5V on purpose. These modules drive their output
rail-to-rail and the ESP32-C3 is not 5V tolerant at 3.6 V absolute max, so a
5V-powered module would overdrive IO3. R7's 5.1k stays in series anyway.
TS3/TS4/TS5 repeat the three signals as solder terminals.

Centred geometry as asked: the LED row has 15.567 mm of headroom at each end,
identical, and the USB-C sits dead centre of the bulge at x=98.0. The module
moved aside to x=115 to make room, which leaves its antenna keep-out facing
the free y=52 edge, 23.9 mm from the nearest LED copper against a rule of 8.

Four screws now: two in the bulge and one at each end of the LED strip, so the
whole length is held rather than just the electronics.

0 DRC errors, 0 unconnected pads, 16 BOM lines, 59 placements, single-sided.

Co-Authored-By: Claude Opus 5 (1M context) <noreply@anthropic.com>
Parts:
- removed J2_1, J3_1: TOUCH_SENSE, symbol Connector:TestPoint
- removed J2_2, J3_2, J4_3: GND, symbol Connector:TestPoint
- removed J4_1: 5V, symbol Connector:TestPoint
- removed J4_2: 3V3, symbol Connector:TestPoint
- removed J4_4: SIG, symbol Connector:TestPoint
- added J4: IO/VCC/GND, symbol Connector:TestPoint
- R10: value 4M7 -> 100k
