File: hardware/ember/ember.kicad_pcb (KiCad board)
At the start: 2 copper layers, 187 x 52 mm, 77 parts, among them J1 USB-C 16P, J4 IO/VCC/GND, Q1 AO3401A, SW1 BOOT, U1 ESP32-C3-MINI-1-N4, U2 SN74AHCT1G125, U3 AP2112K-3.3, U4 USBLC6-2SC6

Commit message: Take the repo URL off the silkscreen
The board will outlive the URL. A repo can move, be renamed or go private,
and a dead link etched into a hundred boards is worse than no link. The
name, revision and copyright stay.

Rebuilt and re-verified: 0 DRC errors, 0 unconnected pads.

Co-Authored-By: Claude Opus 5 (1M context) <noreply@anthropic.com>
Other:
- board text removed: "github.com/fionnf/linked-friend-lights-public"

Commit message: Enforce via hole-to-hole spacing before ordering
The stitching grid and the per-pad ground vias could land 0.45-0.5 mm apart,
at or under JLC hole-to-hole minimum. Two such pairs existed. finish_routing
now drops the later via of any pair closer than 0.75 mm.

0 DRC errors, 0 unconnected pads, gerbers and BOM regenerated.

Co-Authored-By: Claude Opus 5 (1M context) <noreply@anthropic.com>
Routing:
- net GND: vias 149 -> 147
