File: hardware/ember/ember.kicad_pcb (KiCad board)
At the start: 2 copper layers, 187 x 52 mm, 77 parts, among them J1 USB-C 16P, J4 IO/VCC/GND, Q1 AO3401A, SW1 BOOT, U1 ESP32-C3-MINI-1-N4, U2 SN74AHCT1G125, U3 AP2112K-3.3, U4 USBLC6-2SC6

Commit message: Add I2C expansion pads; keep the HRO USB-C after measuring the cheap one
Four solder pads on IO4 and IO10 -- GND / 3V3 / SDA / SCL -- sited directly
above the two GPIOs they serve, in the gap between the regulator row and the
module. Zero placements, zero BOM lines, and whatever sensor turns out to be
wanted later plugs in here instead of needing a board spin.

They started on the far side of the board, which needed a B.Cu jumper running
straight through the antenna keep-out. Moving them beside their own pins made
the runs a few millimetres and the problem disappeared.

The USB-C stays on the HRO TYPE-C-31-M-12 (C165948) despite $0.10 being
available. The cheaper GT-USB-7010ASV looked ideal -- KiCad has a footprint
drawn for that exact part and JLC stocks it, pad naming identical -- but
measured, its own mounting posts sit 0.175 mm from its own GND pads, under
JLC's 0.25 mm hole-to-copper minimum. Not worth a fab flag on the power inlet
for ten cents.

0 DRC errors, 0 unconnected pads, 41 nets, 59 placements.

Co-Authored-By: Claude Opus 5 (1M context) <noreply@anthropic.com>
Parts:
- added I1: I2C_SDA, TestPoint_Pad_D1.0mm, F.Cu at (110.5, 27.3)
- added I2: I2C_SCL, TestPoint_Pad_D1.0mm, F.Cu at (113.0, 27.3)
- added I3: +3V3, TestPoint_Pad_D1.0mm, F.Cu at (108.0, 27.3)
- added I4: GND, TestPoint_Pad_D1.0mm, F.Cu at (105.5, 27.3)
Connections:
- U1 pad 16: (no net) -> I2C_SCL
- U1 pad 18: (no net) -> I2C_SDA
Routing:
- net TOUCH_SENSE: track 38.8 -> 51.8 mm, vias 2 -> 3
- net LED_DATA_3V3: track 45.6 -> 52.4 mm
- net +5V: track 16.6 -> 23.3 mm, vias 0 -> 2
- net UART_TX: track 10.3 -> 16.9 mm, vias 0 -> 2
- net EN: track 47.6 -> 53.9 mm
- net I2C_SDA: track 0.00 -> 6.20 mm
- net TOUCH_GPIO: track 38.6 -> 32.9 mm, vias 0 -> 2
- net I2C_SCL: track 0.00 -> 5.30 mm
- net VBUS_RAW: track 39.9 -> 44.3 mm, vias 2 -> 3
- net VBUS_F: track 26.1 -> 30.4 mm, vias 0 -> 2
- net USB_DP: track 26.1 -> 29.8 mm, vias 2 -> 4
- net CC1: track 13.7 -> 10.2 mm, vias 2 -> 0
- net BOOT_N: track 35.5 -> 38.7 mm, vias 0 -> 2
- net LED_5V: track 43.9 -> 47.0 mm, vias 2 -> 4
- net USB_DP_CONN: track 20.6 -> 17.9 mm
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Other:
- board text added: "I2C GND 3V3 SDA SCL"

Commit message: Put the pad row on a single 2.54 mm pitch
Eight pads sat in one visual row with three different gaps -- 2.5 mm for the
I2C group, 3.0 for the test points, then a 5.0 jump. It read as misaligned
because it was.

The whole row is now 2.54 mm, which is 0.1 inch, so a standard pin header or
a dupont cable actually fits the I2C pads instead of merely being near them.
The TTP223 terminals get the same pitch.

Labels now come from each pad own value field rather than one long silk
string that landed nowhere near the pads it named.

J1 was checked and is genuinely centred: pad midpoint 98.00 against a bulge
centre of 98.00.

0 DRC errors, 0 unconnected pads. Order package regenerated.

Co-Authored-By: Claude Opus 5 (1M context) <noreply@anthropic.com>
Parts:
- moved TP1 8.85 mm to (120.8, 27.3)
- moved TP2 3.77 mm to (118.2, 27.3)
- moved TP3 3.31 mm to (115.7, 27.3)
- moved TP4 2.86 mm to (113.2, 27.3)
- moved I4 2.50 mm to (103.0, 27.3)
- moved I3 2.46 mm to (105.5, 27.3)
- moved I1 2.42 mm to (108.1, 27.3)
- moved I2 2.38 mm to (110.6, 27.3)
- moved TS5 0.92 mm to (104.1, 35.5)
- moved TS4 0.46 mm to (101.5, 35.5)
Routing:
- net +3V3: track 110.4 -> 94.8 mm, vias 5 -> 4
- net VBUS_RAW: track 44.3 -> 59.7 mm, vias 3 -> 2
- net STRAP8: track 23.9 -> 33.1 mm
- net CC2: track 13.6 -> 22.5 mm, vias 0 -> 2
- net UART_TX: track 16.9 -> 9.63 mm, vias 2 -> 0
- net TOUCH_GPIO: track 32.9 -> 39.4 mm
- net VBUS_F: track 30.4 -> 24.2 mm, vias 2 -> 0
- net LED_5V: track 47.0 -> 52.4 mm
- net UART_RX: track 10.7 -> 15.6 mm
- net EN: track 53.9 -> 57.8 mm
- net USB_DM_CONN: track 22.1 -> 25.1 mm, vias 0 -> 2
- net BOOT_N: track 38.7 -> 41.3 mm, vias 2 -> 3
- net +5V: track 23.3 -> 25.9 mm, vias 2 -> 0
- net USB_DP: track 29.8 -> 27.3 mm, vias 4 -> 2
- net I2C_SDA: track 6.20 -> 8.62 mm
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Other:
- board text added: "I2C"
- board text added: "TTP223"
- board text removed: "I2C GND 3V3 SDA SCL"
- board text removed: "TTP223 IO VCC GND"
