File: hardware/ember/ember.kicad_sch (KiCad schematic)
At the start: 70 parts, among them J1 USB-C 16P, J4 IO/VCC/GND, Q1 AO3401A, SW1 BOOT, U1 ESP32-C3-MINI-1-N4, U2 SN74AHCT1G125, U3 AP2112K-3.3, U4 USBLC6-2SC6

Commit message: Add I2C expansion pads; keep the HRO USB-C after measuring the cheap one
Four solder pads on IO4 and IO10 -- GND / 3V3 / SDA / SCL -- sited directly
above the two GPIOs they serve, in the gap between the regulator row and the
module. Zero placements, zero BOM lines, and whatever sensor turns out to be
wanted later plugs in here instead of needing a board spin.

They started on the far side of the board, which needed a B.Cu jumper running
straight through the antenna keep-out. Moving them beside their own pins made
the runs a few millimetres and the problem disappeared.

The USB-C stays on the HRO TYPE-C-31-M-12 (C165948) despite $0.10 being
available. The cheaper GT-USB-7010ASV looked ideal -- KiCad has a footprint
drawn for that exact part and JLC stocks it, pad naming identical -- but
measured, its own mounting posts sit 0.175 mm from its own GND pads, under
JLC's 0.25 mm hole-to-copper minimum. Not worth a fab flag on the power inlet
for ten cents.

0 DRC errors, 0 unconnected pads, 41 nets, 59 placements.

Co-Authored-By: Claude Opus 5 (1M context) <noreply@anthropic.com>
Other:
- company: (c) 2026 Fionn Ferreira - github.com/fionnf/linked-friend-lights-public -> (c) 2026 Fionn Ferreira - github.com/fionnf/ember
Changed lines of the file:
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@@
     (date "2026-08-20")
     (rev "G")
-    (company "(c) 2026 Fionn Ferreira - github.com/fionnf/linked-friend-lights-public")
+    (company "(c) 2026 Fionn Ferreira - github.com/fionnf/ember")
   )
   (symbol (lib_id "Device:C_Polarized") (at 25.4 25.4 0) (unit 1)
@@
     (effects (font (size 1.27 1.27)) (justify left))
 )
+  (wire (pts (xy 815.34 48.26) (xy 819.15 48.26))
+    (stroke (width 0) (type default)))
+  (global_label "I2C_SCL" (shape passive) (at 819.15 48.26 0)
+    (effects (font (size 1.27 1.27)) (justify left))
+)
+  (wire (pts (xy 815.34 33.019999999999996) (xy 819.15 33.019999999999996))
+    (stroke (width 0) (type default)))
+  (global_label "I2C_SDA" (shape passive) (at 819.15 33.019999999999996 0)
+    (effects (font (size 1.27 1.27)) (justify left))
+)
